Commit message: initial commit for demo using xarm6 with xarm gripper and Kinect.

File: k4a_arm_support/urdf/K4A.xacro (robot description, xacro)
@@ -2,5 +2,5 @@
 <robot name="k4a" xmlns:xacro="http://ros.org/wiki/xacro">
   <link name="world"/>
-  <link name="winml_link"/>
+  <link name="ros_msft_onnx_link"/>
   <link name="k4a_link_optical" />
   <link name="table">
@@ -64,7 +64,7 @@
       <origin xyz="1.0 0 0" rpy="0 0 3.14159"/>
   </joint>
-  <joint name="winml_to_k4a_optical" type="fixed">
+  <joint name="ros_msft_onnx_to_k4a_optical" type="fixed">
       <parent link="k4a_link_optical"/>
-      <child link="winml_link"/>
+      <child link="ros_msft_onnx_link"/>
       <origin xyz="0 0 0" rpy="0 0 0"/>
   </joint>

File: k4a_arm_support/urdf/UR3_K4A.xacro (robot description, xacro)
@@ -6,5 +6,5 @@
   <xacro:ur3_robot prefix="" joint_limited="false"/>
   <link name="world"/>
-  <link name="winml_link"/>
+  <link name="ros_msft_onnx_link"/>
   <link name="k4a_link_optical" />
   <link name="table">
@@ -98,7 +98,7 @@
       <origin xyz="0.017 0 0" rpy="0 0 0"/>
   </joint>
-  <joint name="winml_to_k4a_optical" type="fixed">
+  <joint name="ros_msft_onnx_to_k4a_optical" type="fixed">
       <parent link="k4a_link_optical"/>
-      <child link="winml_link"/>
+      <child link="ros_msft_onnx_link"/>
       <origin xyz="-0.035 0 0" rpy="0 0 ${-pi}"/>
   </joint>

File: k4a_arm_support/urdf/UR3_Lifecam.xacro (robot description, xacro)
@@ -6,5 +6,5 @@
   <xacro:ur3_robot prefix="" joint_limited="false"/>
   <link name="world"/>
-  <link name="winml_link"/>
+  <link name="ros_msft_onnx_link"/>
   <link name="k4a_link_optical" />
   <link name="wall1">
@@ -178,7 +178,7 @@
       <origin xyz="0 0 0.02" rpy="0 0 0"/>
   </joint>
-  <joint name="winml_to_k4a_optical" type="fixed">
+  <joint name="ros_msft_onnx_to_k4a_optical" type="fixed">
       <parent link="k4a_link_optical"/>
-      <child link="winml_link"/>
+      <child link="ros_msft_onnx_link"/>
       <origin xyz="0 0 0.027" rpy="0 0 0"/>
   </joint>

File: k4a_arm_support/urdf/workcell.xacro (robot description, xacro)
@@ -6,5 +6,5 @@
   <xacro:ur3_robot prefix="" joint_limited="false"/>
   <link name="world"/>
-  <link name="winml_link"/>
+  <link name="ros_msft_onnx_link"/>
   <link name="k4a_link_optical" />
   <link name="table">
@@ -78,7 +78,7 @@
       <origin xyz="0.017 0 0" rpy="0 0 0"/>
   </joint>
-  <joint name="winml_to_k4a_optical" type="fixed">
+  <joint name="ros_msft_onnx_to_k4a_optical" type="fixed">
       <parent link="k4a_link_optical"/>
-      <child link="winml_link"/>
+      <child link="ros_msft_onnx_link"/>
       <origin xyz="0.04 0 0" rpy="0 0 0"/>
   </joint>
